File: pcb/FreeVision1200/FreeVision1200.kicad_sch (KiCad schematic)
At the start: 0 parts

Commit message: Schematic update
Other:
- added sheet Amiga (amiga.kicad_sch)
- added sheet Audio (audio.kicad_sch)
- added sheet Buffers Addr (buffers2.kicad_sch)
- added sheet Buffers Data (buffers1.kicad_sch)
- added sheet Power (power.kicad_sch)
- added sheet hdmi (hdmi.kicad_sch)
